Commit message: Add files via upload

File: moon/src/urdf/rmoon.urdf (robot description, URDF)
Before this commit: robot moon, 10 links, 9 joints
Links:
- added link base, mass 1; collision box size=0.001 0.5 0.001; visual box size=0.001 0.001 0.001
- added link sonar, mass 1e-5; visual cylinder length=0.01 radius=0.04
- added link sonar2, mass 1e-5; visual cylinder length=0.01 radius=0.04
- added link turn_aft, mass 1
- added link turn_f, mass 1
- link aftbody: geometry collision mesh filename=package://moon/src/meshes/rtbod.stl; visual mesh filename=package://moon/src/meshes/rtbod.stl
- link lmid: geometry collision mesh filename=package://moon/src/meshes/rtmid.stl; visual mesh filename=package://moon/src/meshes/rtmid.stl
Joints:
- removed joint LefttoRight
- added joint LefttoBase: type revolute, parent base, child lmid, origin xyz=0 0 0 rpy=0 0 0, axis 0 1 0 , limit lower=-1.57079632679 upper=1.57079632679 effort=1110 velocity=10
- added joint RighttoBase: type revolute, parent base, child rmid, origin xyz=0 0 0 rpy=0 0 0, axis 0 1 0 , limit lower=-1.57079632679 upper=1.57079632679 effort=1110 velocity=10
- added joint sonar: type fixed, parent forebody, child sonar, origin xyz=0.45 0 0 rpy=0 0 0, axis 0 1 0
- added joint sonar2: type fixed, parent aftbody, child sonar2, origin xyz=-0.45 0 0 rpy=0 0 3.14159265359, axis 0 1 0
- added joint turning_aft: type revolute, parent turn_aft, child aftbody, origin xyz=0 0 0 rpy=0 0 0, axis 1 0 0 , limit lower=-1.57079632679 upper=1.57079632679 effort=500 velocity=10
- added joint turning_f: type revolute, parent turn_f, child forebody, origin xyz=0 0 0 rpy=0 0 0, axis 1 0 0 , limit lower=-1.57079632679 upper=1.57079632679 effort=500 velocity=10
- joint aft: child aftbody -> turn_aft; limit lower=-0.28 upper=0 effort=1000 velocity=1 -> lower=-0.28 upper=0 effort=20000 velocity=10; origin xyz=-0.600000 0 0.020000 rpy=0 0 0 -> xyz=-0.600000 0 0.02 rpy=0 0 0; parent rmid -> lmid
- joint aftLeftTire_j: axis 1 0 0  ->  1 0  0; origin xyz=-0.15 -0.5 -0.025000 rpy=0 0 1.57079632679 -> xyz=-0.15 -0.5 -0.025 rpy=0 0 1.57079632679
- joint aftRightTire_j: axis 1 0 0  ->  1 0  0; origin xyz=-0.15 0.5 -0.025000 rpy=0 0 -1.57079632679 -> xyz=-0.15 0.5 -0.025 rpy=0 0 -1.57079632679
- joint fore: child forebody -> turn_f; limit lower=0 upper=0.28 effort=1000 velocity=1 -> lower=0 upper=0.28 effort=20000 velocity=10; origin xyz=0.600000 0 0.020000 rpy=0 0 0 -> xyz=0.600000 0 0.02 rpy=0 0 0; parent lmid -> rmid
- joint foreLeftTire_j: axis 1 0 0  ->  1 0  0; origin xyz=0.15 -0.5 -0.025000 rpy=0 0 1.57079632679 -> xyz=0.15 -0.5 -0.025 rpy=0 0 1.57079632679
- joint foreRightTire_j: axis 1 0 0  ->  1 0  0; origin xyz=0.15 0.5 -0.025000 rpy=0 0 -1.57079632679 -> xyz=0.15 0.5 -0.025 rpy=0 0 -1.57079632679
- joint midLeftTire_j: axis 1 0 0  ->  1 0  0; origin xyz=0 -0.5 0.005000 rpy=0 0 1.57079632679 -> xyz=0 -0.5 0.005 rpy=0 0 1.57079632679
- joint midRightTire_j: axis 1 0 0  ->  1 0  0; origin xyz=0 0.5 0.005000 rpy=0 0 -1.57079632679 -> xyz=0 0.5 0.005 rpy=0 0 -1.57079632679

Commit message: Add files via upload

File: moon/src/urdf/rmoon.urdf (robot description, URDF)
Before this commit: robot moon, 15 links, 14 joints
Links:
- removed link base
Joints:
- removed joint LefttoBase
- removed joint RighttoBase
- added joint LefttoRight: type revolute, parent lmid, child rmid, origin xyz=0 0 0 rpy=0 0 0, axis 0 1 0 , limit lower=-1.57079632679 upper=1.57079632679 effort=1110 velocity=10
- joint aftLeftTire_j: axis  1 0  0 -> 1 0 0 
- joint aftRightTire_j: axis  1 0  0 -> 1 0 0 
- joint foreLeftTire_j: axis  1 0  0 -> 1 0 0 
- joint foreRightTire_j: axis  1 0  0 -> 1 0 0 
- joint midLeftTire_j: axis  1 0  0 -> 1 0 0 ; parent lmid -> rmid
- joint midRightTire_j: axis  1 0  0 -> 1 0 0 
- joint sonar: origin xyz=0.45 0 0 rpy=0 0 0 -> xyz=0.4 0 0 rpy=0 0 0
- joint sonar2: origin xyz=-0.45 0 0 rpy=0 0 3.14159265359 -> xyz=-0.4 0 0 rpy=0 0 3.14159265359

Commit message: Add files via upload

File: moon/src/urdf/rmoon.urdf (robot description, URDF)
Before this commit: robot moon, 14 links, 13 joints
Links:
- removed link aftLeftTire
- removed link aftRightTire
- removed link foreLeftTire
- removed link foreRightTire
- removed link midLeftTire
- removed link midRightTire
- added link aftLeftWheel, mass 8; collision cylinder length=0.2 radius=0.3; visual mesh filename=package://moon/src/meshes/tire.stl
- added link aftRightWheel, mass 8; collision cylinder length=0.2 radius=0.3; visual mesh filename=package://moon/src/meshes/tire.stl
- added link foreLeftWheel, mass 8; collision cylinder length=0.2 radius=0.3; visual mesh filename=package://moon/src/meshes/tire.stl
- added link foreRightWheel, mass 8; collision cylinder length=0.2 radius=0.3; visual mesh filename=package://moon/src/meshes/tire.stl
- added link midLeftWheel, mass 8; collision cylinder length=0.2 radius=0.3; visual mesh filename=package://moon/src/meshes/tire.stl
- added link midRightWheel, mass 8; collision cylinder length=0.2 radius=0.3; visual mesh filename=package://moon/src/meshes/tire.stl
Joints:
- removed joint aftLeftTire_j
- removed joint aftRightTire_j
- removed joint foreLeftTire_j
- removed joint foreRightTire_j
- removed joint midLeftTire_j
- removed joint midRightTire_j
- added joint aftLeftWheel_j: type continuous, parent aftbody, child aftLeftWheel, origin xyz=-0.15 -0.5 -0.025 rpy=0 0 1.57079632679, axis 1 0 0 , limit effort=1000 velocity=100
- added joint aftRightWheel_j: type continuous, parent aftbody, child aftRightWheel, origin xyz=-0.15 0.5 -0.025 rpy=0 0 -1.57079632679, axis 1 0 0 , limit effort=1000 velocity=100
- added joint foreLeftWheel_j: type continuous, parent forebody, child foreLeftWheel, origin xyz=0.15 -0.5 -0.025 rpy=0 0 1.57079632679, axis 1 0 0 , limit effort=1000 velocity=100
- added joint foreRightWheel_j: type continuous, parent forebody, child foreRightWheel, origin xyz=0.15 0.5 -0.025 rpy=0 0 -1.57079632679, axis 1 0 0 , limit effort=1000 velocity=100
- added joint midLeftWheel_j: type continuous, parent rmid, child midLeftWheel, origin xyz=0 -0.5 0.005 rpy=0 0 1.57079632679, axis 1 0 0 , limit effort=1000 velocity=100
- added joint midRightWheel_j: type continuous, parent rmid, child midRightWheel, origin xyz=0 0.5 0.005 rpy=0 0 -1.57079632679, axis 1 0 0 , limit effort=1000 velocity=100
